File: Board/LightSensor.brd (EAGLE design)
At the start: 100 x 80 mm, 11 parts, among them IC1 74LS07N

Commit message: Rotary sw.
Parts:
- removed SENSOR: (no value), pinhead:2X04
- added JP1: (no value), pinhead:1X04
- added S1: (no value), switch-dil:A1353HEX
Connections:
- new net N$10: ARDUINO.5, S1.1
- new net N$11: ARDUINO.6, S1.2
- new net N$12: ARDUINO.7, S1.4
- new net N$13: ARDUINO.8, S1.8
- net GND: now also JP1.4, S1.C; no longer SENSOR.2, SENSOR.4, SENSOR.6, SENSOR.8
- net N$6: no longer SENSOR.7
- net N$7: now also JP1.3; no longer SENSOR.5
- net N$8: now also JP1.2; no longer SENSOR.3
- net N$9: now also JP1.1; no longer SENSOR.1
Routing:
- net GND: track 90.3 -> 82.1 mm
- net N$8: track 34.9 -> 33.4 mm
Changed lines of the file:
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@@
 <element name="R5" library="resistor" package="0204/5" value="4.7k" x="40.64" y="20.32" rot="R90"/>
 <element name="R6" library="resistor" package="0204/5" value="4.7k" x="38.1" y="20.32" rot="R90"/>
-<element name="SENSOR" library="pinhead" package="2X04" value="" x="41.91" y="6.35"/>
+<element name="JP1" library="pinhead" package="1X04" value="" x="6.35" y="-3.81"/>
+<element name="S1" library="switch-dil" package="A1353HEX" value="" x="-6.35" y="2.54">
+<attribute name="OC_NEWARK" value="unknown" x="-6.35" y="2.54" size="1.778" layer="27" display="off"/>
+<attribute name="MPN" value="" x="-6.35" y="2.54" size="1.778" layer="27" display="off"/>
+<attribute name="MF" value="" x="-6.35" y="2.54" size="1.778" layer="27" display="off"/>
+<attribute name="OC_FARNELL" value="unknown" x="-6.35" y="2.54" size="1.778" layer="27" display="off"/>
+</element>
 </elements>
 <signals>
@@
 <contactref element="MIDIOUT" pad="3"/>
 <contactref element="ARDUINO" pad="23"/>
-<contactref element="SENSOR" pad="8"/>
-<contactref element="SENSOR" pad="6"/>
-<contactref element="SENSOR" pad="4"/>
-<contactref element="SENSOR" pad="2"/>
 <contactref element="PWR" pad="2"/>
 <wire x1="10.287" y1="40.4622" x2="10.287" y2="41.8338" width="0.254" layer="1"/>
@@
 <wire x1="10.287" y1="41.8338" x2="10.16" y2="41.91" width="0.254" layer="1"/>
 <wire x1="20.1168" y1="30.6324" x2="20.32" y2="30.48" width="0.254" layer="1"/>
-<wire x1="40.4622" y1="7.5438" x2="38.1762" y2="7.5438" width="0.254" layer="1"/>
-<wire x1="38.1762" y1="7.5438" x2="38.1" y2="7.62" width="0.254" layer="1"/>
-<wire x1="40.4622" y1="7.5438" x2="40.64" y2="7.62" width="0.254" layer="1"/>
-<wire x1="40.6908" y1="7.5438" x2="42.9768" y2="7.5438" width="0.254" layer="1"/>
-<wire x1="42.9768" y1="7.5438" x2="43.18" y2="7.62" width="0.254" layer="1"/>
-<wire x1="40.6908" y1="7.5438" x2="40.64" y2="7.62" width="0.254" layer="1"/>
 <wire x1="53.2638" y1="15.3162" x2="53.2638" y2="29.0322" width="0.254" layer="16"/>
 <wire x1="45.72" y1="7.7724" x2="51.435" y2="13.4874" width="0.254" layer="16"/>
 <wire x1="51.435" y1="13.4874" x2="53.2638" y2="15.3162" width="0.254" layer="16"/>
 <wire x1="53.2638" y1="29.0322" x2="53.34" y2="29.21" width="0.254" layer="16"/>
-<wire x1="45.72" y1="7.7724" x2="45.72" y2="7.62" width="0.254" layer="16"/>
 <wire x1="51.435" y1="13.4874" x2="59.6646" y2="5.2578" width="0.254" layer="16"/>
 <wire x1="59.6646" y1="5.2578" x2="59.69" y2="5.08" width="0.254" layer="16"/>
-<wire x1="45.72" y1="7.5438" x2="43.2054" y2="7.5438" width="0.254" layer="1"/>
-<wire x1="43.2054" y1="7.5438" x2="43.18" y2="7.62" width="0.254" layer="1"/>
-<wire x1="45.72" y1="7.5438" x2="45.72" y2="7.62" width="0.254" layer="1"/>
 <wire x1="20.3454" y1="29.718" x2="20.3454" y2="30.4038" width="0.254" layer="16"/>
 <wire x1="37.9476" y1="12.1158" x2="20.3454" y2="29.718" width="0.254" layer="16"/>
 <wire x1="37.9476" y1="7.7724" x2="37.9476" y2="12.1158" width="0.254" layer="16"/>
 <wire x1="20.3454" y1="30.4038" x2="20.32" y2="30.48" width="0.254" layer="16"/>
-<wire x1="37.9476" y1="7.7724" x2="38.1" y2="7.62" width="0.254" layer="16"/>
+<contactref element="JP1" pad="4"/>
+<contactref element="S1" pad="C"/>
+<wire x1="37.9476" y1="7.7724" x2="45.72" y2="7.7724" width="0" layer="19" extent="16-16"/>
+<wire x1="10.16" y1="-3.81" x2="37.9476" y2="7.7724" width="0" layer="19" extent="16-16"/>
+<wire x1="-2.54" y1="2.54" x2="10.16" y2="-3.81" width="0" layer="19" extent="1-1"/>
 </signal>
 <signal name="VCC">
@@
 <signal name="N$6">
 <contactref element="R3" pad="1"/>
-<contactref element="SENSOR" pad="7"/>
 <contactref element="ARDUINO" pad="20"/>
 <wire x1="45.72" y1="9.3726" x2="45.72" y2="17.78" width="0.254" layer="1"/>
@@
 <wire x1="46.863" y1="6.4008" x2="46.863" y2="8.2296" width="0.254" layer="1"/>
 <wire x1="45.72" y1="5.2578" x2="46.863" y2="6.4008" width="0.254" layer="1"/>
-<wire x1="45.72" y1="5.2578" x2="45.72" y2="5.08" width="0.254" layer="1"/>
 <wire x1="36.576" y1="22.86" x2="20.32" y2="22.86" width="0.254" layer="1"/>
 <wire x1="38.862" y1="20.574" x2="36.576" y2="22.86" width="0.254" layer="1"/>
@@
 <signal name="N$7">
 <contactref element="R4" pad="1"/>
-<contactref element="SENSOR" pad="5"/>
 <contactref element="ARDUINO" pad="19"/>
 <wire x1="42.9768" y1="9.144" x2="42.9768" y2="17.6022" width="0.254" layer="16"/>
@@
 <wire x1="42.9768" y1="5.2578" x2="42.0624" y2="6.1722" width="0.254" layer="16"/>
 <wire x1="42.9768" y1="17.6022" x2="43.18" y2="17.78" width="0.254" layer="16"/>
-<wire x1="42.9768" y1="5.2578" x2="43.18" y2="5.08" width="0.254" layer="16"/>
 <wire x1="40.6908" y1="20.1168" x2="20.3454" y2="20.1168" width="0.254" layer="1"/>
 <wire x1="42.9768" y1="17.8308" x2="40.6908" y2="20.1168" width="0.254" layer="1"/>
 <wire x1="20.3454" y1="20.1168" x2="20.32" y2="20.32" width="0.254" layer="1"/>
 <wire x1="42.9768" y1="17.8308" x2="43.18" y2="17.78" width="0.254" layer="1"/>
+<contactref element="JP1" pad="3"/>
+<wire x1="7.62" y1="-3.81" x2="20.3454" y2="20.1168" width="0" layer="19" extent="1-1"/>
 </signal>
 <signal name="N$8">
 <contactref element="R5" pad="1"/>
-<contactref element="SENSOR" pad="3"/>
 <contactref element="ARDUINO" pad="18"/>
 <wire x1="40.4622" y1="9.144" x2="40.4622" y2="17.6022" width="0.254" layer="16"/>
 <wire x1="39.5478" y1="8.2296" x2="40.4622" y2="9.144" width="0.254" layer="16"/>
 <wire x1="39.5478" y1="6.1722" x2="39.5478" y2="8.2296" width="0.254" layer="16"/>
-<wire x1="40.64" y1="5.08" x2="39.5478" y2="6.1722" width="0.254" layer="16"/>
 <wire x1="40.4622" y1="17.6022" x2="40.64" y2="17.78" width="0.254" layer="16"/>
 <wire x1="36.576" y1="17.8308" x2="20.3454" y2="17.8308" width="0.254" layer="1"/>
@@
 <wire x1="20.3454" y1="17.8308" x2="20.32" y2="17.78" width="0.254" layer="1"/>
 <wire x1="40.4622" y1="17.8308" x2="40.64" y2="17.78" width="0.254" layer="1"/>
+<contactref element="JP1" pad="2"/>
+<wire x1="5.08" y1="-3.81" x2="20.32" y2="17.78" width="0" layer="19" extent="1-1"/>
 </signal>
 <signal name="N$9">
 <contactref element="R6" pad="1"/>
-<contactref element="SENSOR" pad="1"/>
 <contactref element="ARDUINO" pad="17"/>
 <wire x1="37.9476" y1="9.144" x2="37.9476" y2="15.3162" width="0.254" layer="1"/>
@@
 <wire x1="37.9476" y1="5.2578" x2="36.8046" y2="6.4008" width="0.254" layer="1"/>
 <wire x1="37.9476" y1="17.6022" x2="38.1" y2="17.78" width="0.254" layer="1"/>
-<wire x1="37.9476" y1="5.2578" x2="38.1" y2="5.08" width="0.254" layer="1"/>
 <wire x1="37.9476" y1="15.3162" x2="20.3454" y2="15.3162" width="0.254" layer="1"/>
 <wire x1="20.3454" y1="15.3162" x2="20.32" y2="15.24" width="0.254" layer="1"/>
+<contactref element="JP1" pad="1"/>
+<wire x1="2.54" y1="-3.81" x2="20.32" y2="15.24" width="0" layer="19" extent="1-1"/>
+</signal>
+<signal name="N$10">
+<contactref element="ARDUINO" pad="5"/>
+<contactref element="S1" pad="1"/>
+<wire x1="-2.54" y1="0" x2="5.08" y2="22.86" width="0" layer="19" extent="1-1"/>
+</signal>
+<signal name="N$11">
+<contactref element="ARDUINO" pad="6"/>
+<contactref element="S1" pad="2"/>
+<wire x1="-10.16" y1="5.08" x2="5.08" y2="20.32" width="0" layer="19" extent="1-1"/>
+</signal>
+<signal name="N$12">
+<contactref element="ARDUINO" pad="7"/>
+<contactref element="S1" pad="4"/>
+<wire x1="-2.54" y1="5.08" x2="5.08" y2="17.78" width="0" layer="19" extent="1-1"/>
+</signal>
+<signal name="N$13">
+<contactref element="ARDUINO" pad="8"/>
+<contactref element="S1" pad="8"/>
+<wire x1="-10.16" y1="0" x2="5.08" y2="15.24" width="0" layer="19" extent="1-1"/>
 </signal>
 </signals>

Commit message: Refined.
Parts:
- removed JP1: (no value), pinhead:1X04
- added SENS: (no value), pinhead:1X04
- moved R1 18.3 mm to (41.9, 20.3)
- moved S1 16.5 mm to (8.89, 8.89)
- moved R2 16.3 mm to (44.5, 20.3)
- moved MIDIOUT 14.0 mm to (24.1, 40.6)
- moved ARDUINO 14.0 mm to (26.7, 20.3)
- moved R3 8.89 mm to (54.6, 20.3)
- moved R4 8.89 mm to (52.1, 20.3)
- moved R5 8.89 mm to (49.5, 20.3)
- moved R6 8.89 mm to (47.0, 20.3)
- moved IC1 4.02 mm to (49.5, 34.3)
- moved PWR 2.54 mm to (55.9, 5.08)
Connections:
- net GND: now also SENS.4; no longer JP1.4
- net N$7: now also SENS.3; no longer JP1.3
- net N$8: now also SENS.2; no longer JP1.2
- net N$9: now also SENS.1; no longer JP1.1
Routing:
- net N$5: track 17.6 -> 47.5 mm
- net GND: track 82.1 -> 106.7 mm
- net N$10: track 0.00 -> 19.2 mm
- net N$6: track 41.0 -> 22.4 mm
- net N$11: track 0.00 -> 17.7 mm
- net N$13: track 0.00 -> 17.7 mm
- net N$1: track 35.6 -> 25.0 mm
- net N$12: track 0.00 -> 9.02 mm
- net N$9: track 31.2 -> 24.1 mm
- net N$4: track 20.2 -> 27.0 mm
- net N$2: track 9.85 -> 13.6 mm
- net N$7: track 37.4 -> 33.7 mm
- net N$8: track 33.4 -> 31.0 mm
- net N$3: track 51.1 -> 50.4 mm
