File: Board/LightSensor.sch (EAGLE design)
At the start: 11 parts, among them IC1 74LS07N

Commit message: Rotary sw.
Parts:
- removed SENSOR: (no value), pinhead:PINHD-2X4
- added JP1: (no value), pinhead:PINHD-1X4
- added S1: (no value), switch-dil:A1353HEX
Connections:
- new net N$10: ARDUINO.2, S1.1
- new net N$11: ARDUINO.3, S1.2
- new net N$12: ARDUINO.4, S1.4
- new net N$13: ARDUINO.5, S1.8
- net GND: now also JP1.4, S1.C; no longer SENSOR.2, SENSOR.4, SENSOR.6, SENSOR.8
- net N$6: no longer SENSOR.7
- net N$7: now also JP1.3; no longer SENSOR.5
- net N$8: now also JP1.2; no longer SENSOR.3
- net N$9: now also JP1.1; no longer SENSOR.1
Other:
- note added: "A0: Orange A1: Red A2: Brown GND: Black"
- moved on the sheet: IC1A, MIDIOUT, R1, R2

Commit message: Refined.
Parts:
- renumbered JP1 to SENS
Other:
- note added: "2: Blue 4: Yellow 5: Blue"
- note added: "Vcc: White GND: Black"
- moved on the sheet: PWR
Changed lines of the file:
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@@
 <part name="MIDIOUT" library="pinhead" deviceset="PINHD-1X5" device=""/>
 <part name="SUPPLY1" library="supply2" deviceset="GND" device=""/>
-<part name="SUPPLY2" library="supply2" deviceset="GND" device=""/>
 <part name="PWR" library="pinhead" deviceset="PINHD-1X2" device=""/>
-<part name="SUPPLY4" library="supply2" deviceset="GND" device=""/>
-<part name="JP1" library="pinhead" deviceset="PINHD-1X4" device=""/>
+<part name="SENS" library="pinhead" deviceset="PINHD-1X4" device=""/>
 <part name="SUPPLY5" library="supply2" deviceset="GND" device=""/>
 <part name="S1" library="switch-dil" deviceset="A1353HEX" device=""/>
@@
 A2: Brown
 GND: Black</text>
+<text x="0" y="25.4" size="1.778" layer="91">Vcc: White
+GND: Black</text>
+<text x="152.4" y="27.94" size="1.778" layer="91">2: Blue
+4: Yellow
+5: Blue</text>
 </plain>
 <instances>
@@
 <instance part="MIDIOUT" gate="A" x="147.32" y="33.02"/>
 <instance part="SUPPLY1" gate="GND" x="137.16" y="20.32"/>
-<instance part="SUPPLY2" gate="GND" x="45.72" y="20.32"/>
-<instance part="PWR" gate="G$1" x="12.7" y="27.94"/>
-<instance part="SUPPLY4" gate="GND" x="5.08" y="20.32"/>
-<instance part="JP1" gate="A" x="7.62" y="68.58" rot="R180"/>
+<instance part="PWR" gate="G$1" x="7.62" y="38.1" rot="R180"/>
+<instance part="SENS" gate="A" x="7.62" y="68.58" rot="R180"/>
 <instance part="SUPPLY5" gate="GND" x="17.78" y="20.32"/>
 <instance part="S1" gate="1" x="86.36" y="40.64" rot="R90"/>
@@
 <wire x1="43.18" y1="48.26" x2="43.18" y2="35.56" width="0.1524" layer="91"/>
 <wire x1="43.18" y1="35.56" x2="53.34" y2="35.56" width="0.1524" layer="91"/>
-<wire x1="43.18" y1="35.56" x2="5.08" y2="35.56" width="0.1524" layer="91"/>
-<wire x1="5.08" y1="35.56" x2="5.08" y2="30.48" width="0.1524" layer="91"/>
+<wire x1="43.18" y1="35.56" x2="10.16" y2="35.56" width="0.1524" layer="91"/>
+<junction x="43.18" y="35.56"/>
 <pinref part="PWR" gate="G$1" pin="1"/>
-<wire x1="5.08" y1="30.48" x2="10.16" y2="30.48" width="0.1524" layer="91"/>
-<junction x="43.18" y="35.56"/>
 </segment>
 </net>
@@
 </segment>
 <segment>
+<pinref part="SENS" gate="A" pin="4"/>
+<wire x1="10.16" y1="71.12" x2="17.78" y2="71.12" width="0.1524" layer="91"/>
+<wire x1="17.78" y1="71.12" x2="17.78" y2="38.1" width="0.1524" layer="91"/>
+<pinref part="SUPPLY5" gate="GND" pin="GND"/>
+<pinref part="PWR" gate="G$1" pin="2"/>
+<wire x1="17.78" y1="38.1" x2="17.78" y2="30.48" width="0.1524" layer="91"/>
+<wire x1="17.78" y1="30.48" x2="17.78" y2="22.86" width="0.1524" layer="91"/>
+<wire x1="10.16" y1="38.1" x2="17.78" y2="38.1" width="0.1524" layer="91"/>
+<junction x="17.78" y="38.1"/>
 <pinref part="ARDUINO" gate="G$1" pin="GND@2"/>
-<pinref part="SUPPLY2" gate="GND" pin="GND"/>
-<wire x1="53.34" y1="30.48" x2="45.72" y2="30.48" width="0.1524" layer="91"/>
-<wire x1="45.72" y1="30.48" x2="45.72" y2="22.86" width="0.1524" layer="91"/>
-</segment>
-<segment>
-<pinref part="PWR" gate="G$1" pin="2"/>
-<pinref part="SUPPLY4" gate="GND" pin="GND"/>
-<wire x1="10.16" y1="27.94" x2="5.08" y2="27.94" width="0.1524" layer="91"/>
-<wire x1="5.08" y1="27.94" x2="5.08" y2="22.86" width="0.1524" layer="91"/>
-</segment>
-<segment>
-<pinref part="JP1" gate="A" pin="4"/>
-<wire x1="10.16" y1="71.12" x2="17.78" y2="71.12" width="0.1524" layer="91"/>
-<wire x1="17.78" y1="71.12" x2="17.78" y2="22.86" width="0.1524" layer="91"/>
-<pinref part="SUPPLY5" gate="GND" pin="GND"/>
+<wire x1="53.34" y1="30.48" x2="17.78" y2="30.48" width="0.1524" layer="91"/>
+<junction x="17.78" y="30.48"/>
 </segment>
 <segment>
@@
 <wire x1="25.4" y1="68.58" x2="25.4" y2="63.5" width="0.1524" layer="91"/>
 <wire x1="25.4" y1="63.5" x2="27.94" y2="63.5" width="0.1524" layer="91"/>
-<pinref part="JP1" gate="A" pin="3"/>
+<pinref part="SENS" gate="A" pin="3"/>
 <wire x1="25.4" y1="68.58" x2="10.16" y2="68.58" width="0.1524" layer="91"/>
 </segment>
@@
 <wire x1="45.72" y1="43.18" x2="53.34" y2="43.18" width="0.1524" layer="91"/>
 <junction x="27.94" y="55.88"/>
-<pinref part="JP1" gate="A" pin="2"/>
+<pinref part="SENS" gate="A" pin="2"/>
 <wire x1="22.86" y1="66.04" x2="10.16" y2="66.04" width="0.1524" layer="91"/>
 </segment>
@@
 <pinref part="ARDUINO" gate="G$1" pin="A0"/>
 <junction x="27.94" y="48.26"/>
-<pinref part="JP1" gate="A" pin="1"/>
+<pinref part="SENS" gate="A" pin="1"/>
 <wire x1="20.32" y1="63.5" x2="10.16" y2="63.5" width="0.1524" layer="91"/>
 </segment>
